Commit message: first commit

File: kinova_description/urdf/j2n6s300_standalone.xacro (robot description, xacro)
@@ -15,7 +15,16 @@
 	xmlns:xacro="http://ros.org/wiki/xacro" name="j2n6s300">
   <xacro:include filename="$(find kinova_description)/urdf/j2n6s300.xacro"/>
+  <xacro:include filename="$(find table_board_fix)/urdf/table.urdf.xacro" />
+<!-- joint -->
+ <!--
+  <joint name="robot_fix" type="fixed">
+    <parent link="table" />
+    <child  link="root"  />
+    <origin rpy="0.0 0.0 3.14" xyz="0.0 2 0.0"/>
+  </joint>
+-->
   <link name="root">
     <visual>
-      <origin xyz="0 0 0" rpy="0 0 0" />
+      <origin xyz="0 5 0" rpy="0 0 0" />
       <geometry>
         <box size = "0.01 0.01 0.01"/>
@@ -34,5 +43,5 @@
   <joint name="connect_root_and_world" type="fixed">
     <child link="root" />
-    <parent link="world" />
+    <parent link="table" />
     <origin xyz="0 0 0" rpy="0 0 0" />
   </joint>

File: kinova_description/urdf/kinova_common.xacro (robot description, xacro)
@@ -57,8 +57,8 @@
         <type>transmission_interface/SimpleTransmission</type>
         <joint name="${joint_name}">
-          <hardwareInterface>hardware_interface/EffortJointInterface</hardwareInterface>
+          <hardwareInterface>EffortJointInterface</hardwareInterface>
         </joint>
         <actuator name="${joint_name}_actuator">
-          <hardwareInterface>hardware_interface/EffortJointInterface</hardwareInterface>
+          <hardwareInterface>EffortJointInterface</hardwareInterface>
         <mechanicalReduction>160</mechanicalReduction>
         </actuator>
@@ -101,8 +101,8 @@
 					<type>transmission_interface/SimpleTransmission</type>
 					<joint name="${prefix}joint_finger_${finger_number}">
-					  <hardwareInterface>hardware_interface/EffortJointInterface</hardwareInterface>
+					  <hardwareInterface>EffortJointInterface</hardwareInterface>
 					</joint>
 					<actuator name="${prefix}joint_finger_${finger_number}_actuator">
-					<hardwareInterface>hardware_interface/EffortJointInterface</hardwareInterface>
+					<hardwareInterface>EffortJointInterface</hardwareInterface>
 					<mechanicalReduction>1</mechanicalReduction>
 					</actuator>
