Commit message: 检查修改

File: kinova_description/objects/objects.urdf.xacro (robot description, xacro)
@@ -2,5 +2,4 @@
 <robot xmlns:xacro="http://ros.org/wiki/xacro"
        name="kinova_sim" >
-<property name="pi" value="3.14159265"/>
 <link
     name="left_basket">

File: kinova_description/urdf/kinova_common.xacro (robot description, xacro)
@@ -57,8 +57,8 @@
         <type>transmission_interface/SimpleTransmission</type>
         <joint name="${joint_name}">
-          <hardwareInterface>EffortJointInterface</hardwareInterface>
+          <hardwareInterface>hardware_interface/EffortJointInterface</hardwareInterface>
         </joint>
         <actuator name="${joint_name}_actuator">
-          <hardwareInterface>EffortJointInterface</hardwareInterface>
+          <hardwareInterface>hardware_interface/EffortJointInterface</hardwareInterface>
         <mechanicalReduction>160</mechanicalReduction>
         </actuator>
@@ -101,8 +101,8 @@
 					<type>transmission_interface/SimpleTransmission</type>
 					<joint name="${prefix}joint_finger_${finger_number}">
-					  <hardwareInterface>EffortJointInterface</hardwareInterface>
+					  <hardwareInterface>hardware_interface/EffortJointInterface</hardwareInterface>
 					</joint>
 					<actuator name="${prefix}joint_finger_${finger_number}_actuator">
-					<hardwareInterface>EffortJointInterface</hardwareInterface>
+					<hardwareInterface>hardware_interface/EffortJointInterface</hardwareInterface>
 					<mechanicalReduction>1</mechanicalReduction>
 					</actuator>

File: kinova_description/urdf/kinova_sim.xacro (robot description, xacro)
@@ -2,5 +2,4 @@
 <robot xmlns:xacro="http://ros.org/wiki/xacro"
        name="kinova_sim" >
-<property name="pi" value="3.14159265"/>
   <!-- include urdf -->
   <xacro:include filename="$(find kinova_description)/urdf/j2s7s300_standalone.xacro" />

File: test_d435_camera.urdf.sim.xacro (robot description, xacro)
@@ -3,5 +3,5 @@
   <xacro:include filename="$(find realsense2_camera)/urdf/_d435.urdf.xacro"/>
   <sensor_d435 parent="tools2">
-    <origin xyz="-0.01 -0.435 0.015" rpy="1.5707963 0 3.1415926"/>
+    <origin xyz="-0.01 -0.405 0.015" rpy="1.5707963 0 3.1415926"/>
   </sensor_d435>
   <link
@@ -51,5 +51,5 @@
     type="fixed">
     <origin
-      xyz="-0.0323 -0.040 -0.5"
+      xyz="-0.0323 -0.050 -0.5"
       rpy="-1.5707963 0 0" />
     <parent
@@ -109,5 +109,5 @@
     type="fixed">
     <origin
-      xyz="0.016 -0.5 -0.48"
+      xyz="0.016 -0.5 -0.49"
       rpy="-1.5707963 0 -1.5707963" />
     <parent

Commit message: (未完成)模型修改,PID参数调节,详见日志

File: kinova_description/objects/objects.urdf.xacro (robot description, xacro)
@@ -112,54 +112,3 @@
       xyz="0 0 0" />
 </joint>
-<!--
-<link
-    name="cone">
-    <inertial>
-      <origin
-        xyz="0 0 0"
-        rpy="0 0 0" />
-      <mass
-        value="1.1E-5" />
-      <inertia
-        ixx="1.1E-5"
-        ixy="1.1E-5"
-        ixz="1.1E-5"
-        iyy="1.1E-5"
-        iyz="1.1E-5"
-        izz="1.1E-5" />
-    </inertial>
-    <visual>
-      <geometry>
-        <mesh
-          filename="$(find kinova_description)/objects/objects/cone.dae" />
-      </geometry>
-    </visual>
-    <material
-        name="">
-        <color
-          rgba="1 1 1 1" />
-        <texture
-          filename="$(find kinova_description)/objects/textures/green.jpg" />
-    </material>
-    <collision>
-      <geometry>
-        <mesh
-          filename="$(find kinova_description)/objects/objects/cone.dae" />
-      </geometry>
-    </collision>
-</link>
-<joint
-    name="cone"
-    type="gearbox">
-    <origin
-      xyz="0 0 0"
-      rpy="0 0 0" />
-    <parent
-      link="right_board" />
-    <child
-      link="cone" />
-    <axis
-      xyz="0 0 0" />
-</joint>
- -->
 </robot>

File: kinova_description/urdf/kinova_sim.xacro (robot description, xacro)
@@ -2,7 +2,7 @@
 <robot xmlns:xacro="http://ros.org/wiki/xacro"
        name="kinova_sim" >
-  <!-- include urdf -->
   <xacro:include filename="$(find kinova_description)/urdf/j2s7s300_standalone.xacro" />
   <xacro:include filename="$(find kinova_description)/objects/objects.urdf.xacro" />
-  <xacro:include filename="$(find realsense2_camera)/urdf/test_d435_camera.urdf.sim.xacro"/>
+  <xacro:include filename="$(find realsense2_camera)/urdf/_d435.urdf.xacro"/>
+  <xacro:include filename="$(find kinova_description)/objects/tools.urdf.xacro" />
 </robot>

Commit message: modify models

File: kinova_description/objects/objects.urdf.xacro (robot description, xacro)
@@ -2,113 +2,165 @@
 <robot xmlns:xacro="http://ros.org/wiki/xacro"
        name="kinova_sim" >
-<link
-    name="left_basket">
-    <inertial>
-      <origin
-        xyz="0 0.5 0"
-        rpy="0 0 0" />
-      <mass
-        value="2.0243" />
-      <inertia
-        ixx="0.031947"
-        ixy="-6.6313E-18"
-        ixz="-2.4676E-18"
-        iyy="0.023762"
-        iyz="-7.8627E-18"
-        izz="0.052372" />
-    </inertial>
-    <visual>
-      <origin
-        xyz="0 0.5 0"
-        rpy="0 0 0" />
-      <geometry>
-        <mesh
-          filename="$(find kinova_description)/objects/meshes/left_basket.dae" />
-      </geometry>
-      <material
-        name="">
-        <color
-          rgba="1 1 1 1" />
-        <texture
-          filename="$(find kinova_description)/objects//textures/blue.jpg" />
-      </material>
-    </visual>
-    <collision>
-      <origin
-        xyz="0 0.5 0"
-        rpy="0 0 0" />
-      <geometry>
-        <mesh
-          filename="$(find kinova_description)/objects/meshes/left_basket.dae" />
-      </geometry>
-    </collision>
+<!-- define the table and baskets-->
+<link name="table">
+  <inertial>
+    <origin
+      xyz="0 0 0"
+      rpy="0 0 0" />
+    <mass
+      value="81.416" />
+    <inertia
+      ixx="17.674"
+      ixy="-4.3368E-16"
+      ixz="4.9467E-16"
+      iyy="17.674"
+      iyz="1.3081E-17"
+      izz="19.456" />
+  </inertial>
+  <visual>
+    <origin
+      xyz="0 0 0"
+      rpy="0 0 0" />
+    <geometry>
+      <mesh
+        filename="package://table_basket_new/meshes/table.STL" />
+    </geometry>
+    <material
+      name="">
+      <color
+        rgba="1 1 1 1" />
+      <texture
+        filename="package://table_basket_new/textures/table_color.jpg" />
+    </material>
+  </visual>
+  <collision>
+    <origin
+      xyz="0 0 0"
+      rpy="0 0 0" />
+    <geometry>
+      <mesh
+        filename="package://table_basket_new/meshes/table.STL" />
+    </geometry>
+  </collision>
 </link>
-<link
-    name="right_board">
-    <inertial>
-      <origin
-        xyz="0 0.5 0"
-        rpy="0 0 0" />
-      <mass
-        value="2.0243" />
-      <inertia
-        ixx="0.023049"
-        ixy="-7.5343E-18"
-        ixz="-5.8775E-36"
-        iyy="0.042"
-        iyz="0"
-        izz="0.06503" />
-    </inertial>
-    <visual>
-      <origin
-        xyz="0 0.5 0"
-        rpy="0 0 0" />
-      <geometry>
-        <mesh
-          filename="$(find kinova_description)/objects/meshes/right_board.dae" />
-      </geometry>
-      <material
-        name="">
-        <color
-          rgba="1 1 1 1" />
-        <texture
-          filename="$(find kinova_description)/objects/textures/green.jpg" />
-      </material>
-    </visual>
-    <collision>
-      <origin
-        xyz="0 0.5 0"
-        rpy="0 0 0" />
-      <geometry>
-        <mesh
-          filename="$(find kinova_description)/objects/meshes/right_board.dae" />
-      </geometry>
-    </collision>
+<link name="left_basket">
+  <inertial>
+    <origin
+      xyz="-1.1102E-16 0 0.031586"
+      rpy="0 0 0" />
+    <mass
+      value="18.812" />
+    <inertia
+      ixx="0.029288"
+      ixy="-2.2695E-18"
+      ixz="-2.6278E-18"
+      iyy="0.01841"
+      iyz="2.5457E-20"
+      izz="0.04459" />
+  </inertial>
+  <visual>
+    <origin
+      xyz="0 0 0"
+      rpy="0 0 0" />
+    <geometry>
+      <mesh
+        filename="package://table_basket_new/meshes/left_basket.STL" />
+    </geometry>
+    <material
+      name="">
+      <color
+        rgba="1 1 1 1" />
+      <texture
+        filename="package://table_basket_new/textures/blue.jpg" />
+    </material>
+  </visual>
+  <collision>
+    <origin
+      xyz="0 0 0"
+      rpy="0 0 0" />
+    <geometry>
+      <mesh
+        filename="package://table_basket_new/meshes/left_basket.STL" />
+    </geometry>
+  </collision>
 </link>
 <joint
-    name="left_fixed"
-    type="fixed">
+  name="left_fix"
+  type="fixed">
+  <origin
+    xyz="0.27 0.275 0"
+    rpy="0 0 0" />
+  <parent
+    link="table" />
+  <child
+    link="left_basket" />
+  <axis
+    xyz="0 0 0" />
+</joint>
+<link name="right_basket">
+  <inertial>
     <origin
-      xyz="0.295 -0.12542 0.008"
+      xyz="0 -5.5511E-17 0.031586"
       rpy="0 0 0" />
-    <parent
-      link="world" />
-    <child
-      link="left_basket" />
-    <axis
-      xyz="0 0 0" />
+    <mass
+      value="18.812" />
+    <inertia
+      ixx="0.029288"
+      ixy="1.3977E-18"
+      ixz="-3.7403E-18"
+      iyy="0.01841"
+      iyz="-5.7134E-19"
+      izz="0.04459" />
+  </inertial>
+  <visual>
+    <origin
+      xyz="0 0 0"
+      rpy="0 0 0" />
+    <geometry>
+      <mesh
+        filename="package://table_basket_new/meshes/right_basket.STL" />
+    </geometry>
+    <material
+      name="">
+      <color
+        rgba="1 1 1 1" />
+      <texture
+        filename="package://table_basket_new/textures/green.jpg" />
+    </material>
+  </visual>
+  <collision>
+    <origin
+      xyz="0 0 0"
+      rpy="0 0 0" />
+    <geometry>
+      <mesh
+        filename="package://table_basket_new/meshes/right_basket.STL" />
+    </geometry>
+  </collision>
+</link>
+<joint
+  name="right_fix"
+  type="fixed">
+  <origin
+    xyz="-0.27 0.275 0"
+    rpy="0 0 0" />
+  <parent
+    link="table" />
+  <child
+    link="right_basket" />
+  <axis
+    xyz="0 0 0" />
 </joint>
-<joint
-    name="right_fixed"
-    type="fixed">
-    <origin
-      xyz="-0.17 -0.10042 0.008"
-      rpy="0 0 0" />
-    <parent
-      link="world" />
-    <child
-      link="right_board" />
-    <axis
-      xyz="0 0 0" />
+<link name="map" />
+<joint name="world_joint" type="fixed">
+  <parent link="map" />
+  <child link = "table" />
+  <origin xyz="0.0 0.0 1.1" rpy="0.0 0.0 0.0" />
+</joint>
+<!-- joint -->
+<joint name="robot_fix" type="fixed">
+  <parent link="table" />
+  <child link = "root" />
+  <origin rpy="0.0 0.0 0.0" xyz="0.0 -0.3 0.0"/>
 </joint>
 </robot>

File: kinova_description/objects/tools.urdf.xacro (robot description, xacro)
@@ -8,4 +8,5 @@
   <link
     name="tools1">
+     <static>true</static>
     <inertial>
       <origin
@@ -13,12 +14,12 @@
         rpy="0 0 0" />
       <mass
-        value="2.0243E-6" />
+        value="2.0243E-24" />
       <inertia
-        ixx="0.031947E-6"
+        ixx="0.031947E-24"
         ixy="-6.6313E-24"
         ixz="-2.4676E-24"
-        iyy="0.023762E-6"
+        iyy="0.023762E-24"
         iyz="-7.8627E-24"
-        izz="0.052372E-6" />
+        izz="0.052372E-24" />
     </inertial>
     <visual>
@@ -43,6 +44,5 @@
         rpy="0 0 0" />
       <geometry>
-        <mesh
-          filename="$(find kinova_description)/objects/tools/first.STL" />
+        <cylinder length="0.01" radius="0.01"/>
       </geometry>
     </collision>
@@ -68,12 +68,12 @@
         rpy="0 0 0" />
       <mass
-        value="2.0243E-6" />
+        value="2.0243E-24" />
       <inertia
-        ixx="0.031947E-6"
+        ixx="0.031947E-24"
         ixy="-6.6313E-24"
         ixz="-2.4676E-24"
-        iyy="0.023762E-6"
+        iyy="0.023762E-24"
         iyz="-7.8627E-24"
-        izz="0.052372E-6" />
+        izz="0.052372E-24" />
     </inertial>
     <visual>

File: kinova_description/urdf/j2s7s300_standalone.xacro (robot description, xacro)
@@ -3,33 +3,18 @@
 <robot xmlns:xi="http://www.w3.org/2001/XInclude"
 	xmlns:gazebo="http://playerstage.sourceforge.net/gazebo/xmlschema/#gz"
-	xmlns:model="http://playerstage.sourceforge.net/gazebo/xmlschema/#model"
+    xmlns:model="http://playerstage.sourceforge.net/gazebo/xmlschema/#model"
 	xmlns:sensor="http://playerstage.sourceforge.net/gazebo/xmlschema/#sensor"
 	xmlns:body="http://playerstage.sourceforge.net/gazebo/xmlschema/#body"
-	xmlns:geom="http://playerstage.sourceforge.net/gazebo/xmlschema/#geom"
-	xmlns:joint="http://playerstage.sourceforge.net/gazebo/xmlschema/#joint"
+    xmlns:geom="http://playerstage.sourceforge.net/gazebo/xmlschema/#geom"
+    xmlns:joint="http://playerstage.sourceforge.net/gazebo/xmlschema/#joint"
 	xmlns:controller="http://playerstage.sourceforge.net/gazebo/xmlschema/#controller"
 	xmlns:interface="http://playerstage.sourceforge.net/gazebo/xmlschema/#interface"
 	xmlns:rendering="http://playerstage.sourceforge.net/gazebo/xmlschema/#rendering"
-	xmlns:renderable="http://playerstage.sourceforge.net/gazebo/xmlschema/#renderable"
-	xmlns:physics="http://playerstage.sourceforge.net/gazebo/xmlschema/#physics"
+    xmlns:renderable="http://playerstage.sourceforge.net/gazebo/xmlschema/#renderable"
+    xmlns:physics="http://playerstage.sourceforge.net/gazebo/xmlschema/#physics"
 	xmlns:xacro="http://ros.org/wiki/xacro" name="j2s7s300">
   <xacro:include filename="$(find kinova_description)/urdf/j2s7s300.xacro"/>
-  <link name="root">
-    <visual>
-      <origin xyz="0 0 0" rpy="0 0 0" />
-      <geometry>
-        <box size = "0.01 0.01 0.01"/>
-      </geometry>
-    <!--<material name="Black" /> -->
-    </visual>
-    <collision>
-      <origin xyz="0 0 0" rpy="0 0 0" />
-      <geometry>
-        <box size = "0.01 0.01 0.01"/>
-      </geometry>
-    </collision>
-  </link>
-  <!-- for gazebo -->
-  <link name="world"/>
+    <link name="root"/>
+    <link name="world"/>
   <joint name="connect_root_and_world" type="fixed">
     <child link="root" />
@@ -37,5 +22,5 @@
     <origin xyz="0 0 0" rpy="0 0 0" />
   </joint>
-  <xacro:property name="robot_root" value="root" />
+  <property name="robot_root" value="root" />
   <xacro:j2s7s300  base_parent="${robot_root}"/>
 </robot>

File: kinova_description/urdf/kinova_sim.xacro (robot description, xacro)
@@ -3,5 +3,4 @@
        name="kinova_sim" >
   <xacro:include filename="$(find kinova_description)/urdf/j2s7s300_standalone.xacro" />
-  <xacro:include filename="$(find kinova_description)/objects/objects.urdf.xacro" />
   <xacro:include filename="$(find realsense2_camera)/urdf/_d435.urdf.xacro"/>
   <xacro:include filename="$(find kinova_description)/objects/tools.urdf.xacro" />
