Commit message: 仿真调试,模型更改(expo)

File: kinova_description/objects/tools.urdf.xacro (robot description, xacro)
@@ -11,5 +11,5 @@
     <inertial>
       <origin
-        xyz="0 0 0"
+        xyz="0.1 0 0"
         rpy="0 0 0" />
       <mass
@@ -44,5 +44,5 @@
         rpy="0 0 0" />
       <geometry>
-        <cylinder length="0.01" radius="0.01"/>
+        <cylinder length="0.001" radius="0.001"/>
       </geometry>
     </collision>

File: kinova_description/urdf/j2s7s300_standalone.xacro (robot description, xacro)
@@ -15,12 +15,13 @@
 	xmlns:xacro="http://ros.org/wiki/xacro" name="j2s7s300">
   <xacro:include filename="$(find kinova_description)/urdf/j2s7s300.xacro"/>
-    <link name="root"/>
-    <link name="world"/>
-  <joint name="connect_root_and_world" type="fixed">
-    <child link="root" />
-    <parent link="world" />
-    <origin xyz="0 0 0" rpy="0 0 0" />
-  </joint>
-  <property name="robot_root" value="root" />
-  <xacro:j2s7s300  base_parent="${robot_root}"/>
+<link name="root"/>
+<!-- for gazebo -->
+<link name="world"/>
+<joint name="connect_root_and_world" type="fixed">
+  <child link="root" />
+  <parent link="world" />
+  <origin xyz="0 0 0" rpy="0 0 0" />
+</joint>
+<xacro:property name="robot_root" value="root" />
+<xacro:j2s7s300  base_parent="${robot_root}"/>
 </robot>

File: kinova_description/urdf/kinova_sim.xacro (robot description, xacro)
@@ -4,4 +4,4 @@
   <xacro:include filename="$(find kinova_description)/urdf/j2s7s300_standalone.xacro" />
   <xacro:include filename="$(find realsense2_camera)/urdf/_d435.urdf.xacro"/>
-  <xacro:include filename="$(find kinova_description)/objects/tools.urdf.xacro" />
+  <xacro:include filename="$(find kinova_description)/objects/tools.urdf.xacro"/>
 </robot>
